Commit message: Fixed error

File: open_manipulator_description/ros2_control/baram.ros2_control.xacro (robot description, xacro)
@@ -143,4 +143,5 @@
         <state_interface name="Present Position"/>
         <state_interface name="Present Velocity"/>
+        <param name="[unit info]">Present Position,0.0015339807878856412,rad,signed,1.35840734641;Goal Position,0.0015339807878856412,rad,signed,1.35840734641;Present Velocity,0.0239691227,rad/s,signed,0.0;Goal Velocity,0.0239691227,rad/s,signed,0.0</param>
         <param name="Operating Mode">3</param>
         <param name="Return Delay Time">0</param>

File: open_manipulator_description/urdf/baram_manipulator/baram_arm.urdf.xacro (robot description, xacro)
@@ -107,5 +107,5 @@
       <child link="${prefix}link4"/>
       <axis xyz="0 0 1"/>
-      <limit effort="10.0" velocity="1.5" lower="-1.57" upper="1.57"/>
+      <limit effort="10.0" velocity="1.5" lower="-1.5707963267948966" upper="1.5707963267948966"/>
       <dynamics damping="0.0"/>
     </joint>
@@ -143,5 +143,5 @@
       <child link="${prefix}link6"/>
       <axis xyz="0 1 0"/>
-      <limit effort="10.0" velocity="1.5" lower="-1.57" upper="1.57"/>
+      <limit effort="10.0" velocity="1.5" lower="-1.5707963267948966" upper="1.5707963267948966"/>
       <dynamics damping="0.0"/>
     </joint>
@@ -167,5 +167,5 @@
       <child link="${prefix}hand"/>
       <axis xyz="0 0 1"/>
-      <limit effort="10.0" velocity="1.5" lower="-1.57" upper="1.57"/>
+      <limit effort="10.0" velocity="1.5" lower="-1.5707963267948966" upper="1.5707963267948966"/>
       <dynamics damping="0.0"/>
     </joint>
